Commit message: change color

File: xacro/modelc.xacro (robot description, xacro)
@@ -8,6 +8,6 @@
                 <box size="0.600 0.400 0.050"/>
             </geometry>
-            <material name="grey">
-                <color rgba="0.5 0.5 0.5 1.0"/>
+            <material name="green">
+                <color rgba="0 1.0 0 1.0"/>
             </material>
         </visual>
@@ -40,6 +40,6 @@
                 <box size="0.250 0.260 0.050"/>
             </geometry>
-            <material name="grey">
-                <color rgba="0.5 0.5 0.5 1.0"/>
+            <material name="red">
+                <color rgba="1.0 0 0 1.0"/>
             </material>
         </visual>
@@ -63,5 +63,7 @@
             </geometry>
             <origin xyz="0 0 0" rpy="0 0 0" />
-            <material name="black" />
+            <material name="black">
+                <color rgba="0 0 0 1.0"/>
+            </material>
         </visual>
         <collision>
@@ -94,5 +96,7 @@
                 <cylinder length="0.05" radius="0.1325"/>
             </geometry>
-            <material name="black" />
+            <material name="black">
+                <color rgba="0 0 0 1.0"/>
+            </material>
         </visual>
         <inertial>
@@ -118,5 +122,7 @@
                 <cylinder length="0.05" radius="0.1325"/>
             </geometry>
-            <material name="black" />
+            <material name="black">
+                <color rgba="0 0 0 1.0"/>
+            </material>
         </visual>
         <inertial>
@@ -144,5 +150,7 @@
                 <cylinder length="0.05" radius="0.1325"/>
             </geometry>
-            <material name="black" />
+            <material name="black">
+                <color rgba="0 0 0 1.0"/>
+            </material>
         </visual>
         <inertial>
